File: kicad/lcd.kicad_sch (KiCad schematic)
At the start: 3 parts, among them J501 Conn_01x13

Commit message: changed from rp2040 to nrf
Other:
- note added: "Max Power Consumption: 32mA w backlight"
- note added: "https://lcsc.com/datasheet/lcsc_datasheet_2410121611_Newvisio-N096-1608TBBIG11-H13_C2890616.pdf"
Changed lines of the file:
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@@
 		(rev "1")
+	)
+	(text "Max Power Consumption: 32mA w backlight"
+		(exclude_from_sim no)
+		(at 121.412 129.032 0)
+		(effects
+			(font
+				(size 1.27 1.27)
+			)
+		)
 	)
 	(text "FPC Connector for LCD\nDatasheet: https://www.seacomp.com/sites/default/files/datasheets/DT010ATFT-Rev1_2-Displaytech-Spec.pdf"
 		(exclude_from_sim no)
 		(at 149.86 73.66 0)
+		(effects
+			(font
+				(size 1.27 1.27)
+			)
+		)
+	)
+	(text "https://lcsc.com/datasheet/lcsc_datasheet_2410121611_Newvisio-N096-1608TBBIG11-H13_C2890616.pdf"
+		(exclude_from_sim no)
+		(at 152.654 132.842 0)
 		(effects
 			(font
@@
 		(dnp no)
 		(fields_autoplaced yes)
-		(property "Reference" "#PWR0504"
+		(property "Reference" "#PWR504"
 			(at 139.7 128.27 0)
 			(effects
@@
 			(project "pocketboard"
 				(path "/bbf42bb3-a553-455a-82cc-5281935de3af/436c300b-cf41-4d3c-817a-13458950e75f"
-					(reference "#PWR0504")
+					(reference "#PWR504")
 					(unit 1)
 				)
@@
 		(dnp no)
 		(fields_autoplaced yes)
-		(property "Reference" "#PWR0501"
+		(property "Reference" "#PWR501"
 			(at 139.7 115.57 0)
 			(effects
@@
 			(project "pocketboard"
 				(path "/bbf42bb3-a553-455a-82cc-5281935de3af/436c300b-cf41-4d3c-817a-13458950e75f"
-					(reference "#PWR0501")
+					(reference "#PWR501")
 					(unit 1)
 				)
@@
 		(dnp no)
 		(fields_autoplaced yes)
-		(property "Reference" "#PWR0502"
+		(property "Reference" "#PWR502"
 			(at 182.88 120.65 0)
 			(effects
@@
 			(project ""
 				(path "/bbf42bb3-a553-455a-82cc-5281935de3af/436c300b-cf41-4d3c-817a-13458950e75f"
-					(reference "#PWR0502")
+					(reference "#PWR502")
 					(unit 1)
 				)
@@
 		(dnp no)
 		(fields_autoplaced yes)
-		(property "Reference" "#PWR0503"
+		(property "Reference" "#PWR503"
 			(at 111.76 128.27 0)
 			(effects
@@
 			(project "pocketboard"
 				(path "/bbf42bb3-a553-455a-82cc-5281935de3af/436c300b-cf41-4d3c-817a-13458950e75f"
-					(reference "#PWR0503")
+					(reference "#PWR503")
 					(unit 1)
 				)

Commit message: board routed
Parts:
- J501: now not fitted; now left out of the parts list
Changed lines of the file:
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@@
 		(unit 1)
 		(exclude_from_sim no)
-		(in_bom yes)
+		(in_bom no)
 		(on_board yes)
-		(dnp no)
+		(dnp yes)
 		(fields_autoplaced yes)
 		(property "Reference" "J501"
