File: kicad/pocketboard.kicad_pcb (KiCad board)
At the start: 4 copper layers, 104.9 x 72.7 mm, 134 parts, among them J1 USB_C_Receptacle_USB2.0_16P, J301 DEBUG_HEADER, J501 Conn_01x13, Q301 2N7002, SW401 SW_Push_Dual, SW402 SW_Push_Dual, SW403 SW_Push_Dual, SW404 SW_Push_Dual, SW405 SW_Push_Dual, SW406 SW_Push_Dual, SW407 SW_Push_Dual, SW408 SW_Push_Dual, SW409 SW_Push_Dual, SW410 SW_Push_Dual, SW411 SW_Push_Dual, SW412 SW_Push_Dual, SW413 SW_Push_Dual, SW414 SW_Push_Dual, SW415 SW_Push_Dual, SW416 SW_Push_Dual, SW417 SW_Push_Dual, SW418 SW_Push_Dual, SW419 SW_Push_Dual, SW420 SW_Push_Dual, SW421 SW_Push_Dual, SW422 SW_Push_Dual, SW423 SW_Push_Dual, SW424 SW_Push_Dual, SW425 SW_Push_Dual, SW426 SW_Push_Dual, SW427 SW_Push_Dual, SW428 SW_Push_Dual, SW429 SW_Push_Dual, SW430 SW_Push_Dual, SW431 SW_Push_Dual, SW432 SW_Push_Dual, SW433 SW_Push_Dual, SW434 SW_Push_Dual, SW435 SW_Push_Dual, SW436 SW_Push_Dual, SW501 SW_Push_45deg, U201 NCP1117-3.3_SOT223, U301 RP2040, U302 W25Q128JVS, Y301 12MHz 20pF

Commit message: changed from rp2040 to nrf
Parts:
- removed D1, D2, D3: D_Zener, Diode_SMD:D_SOD-923
- removed D301, D302, D303, D304, D305, D306, D307, D308, D309, D310: LED, LED_SMD:LED_0603_1608Metric
- removed D401, D402, D403, D404, D405, D406, D407, D408, D409, D410, D411, D412, D413, D414, D415, D416, D417, D418, D419, D420, D421, D422, D423, D424, D425, D426, D427, D428, D429, D430, D431, D432, D433, D434, D435, D436: D, Diode_SMD:D_SOD-123
- removed Q301: 2N7002, Package_TO_SOT_SMD:SOT-23
- removed R304, R305, R306, R307, R308, R309, R310, R311, R312, R313: 33R, Resistor_SMD:R_0402_1005Metric
- removed R314: 1k, Resistor_SMD:R_0402_1005Metric
- removed R315, R316: 5k1, Resistor_SMD:R_0603_1608Metric
- removed SW501: SW_Push_45deg, Button_Switch_SMD:SW_Push_1P1T_XKB_TS-1187A
- removed U302: W25Q128JVS, Package_SO:SOIC-8_5.23x5.23mm_P1.27mm
- added C203: 10u, Capacitor_SMD:C_0402_1005Metric, F.Cu at (137.0, 40.8)
- added C204: 10u, Capacitor_SMD:C_0402_1005Metric, F.Cu at (138.6, 43.3)
- added C205: 10u, Capacitor_SMD:C_0402_1005Metric, B.Cu at (127.2, 84.0)
- added C315: 1p, Capacitor_SMD:C_0402_1005Metric, F.Cu at (121.3, 52.6)
- added C316: 1p, Capacitor_SMD:C_0402_1005Metric, F.Cu at (121.3, 48.4)
- added C317: 1p5, Capacitor_SMD:C_0402_1005Metric, F.Cu at (120.6, 46.6)
- added C318: 10u, Capacitor_SMD:C_0402_1005Metric, F.Cu at (138.6, 45.4)
- added C319: 1u, Capacitor_SMD:C_0402_1005Metric, F.Cu at (130.0, 60.2)
- added C320: 1u, Capacitor_SMD:C_0402_1005Metric, F.Cu at (134.0, 60.2)
- added D311: LED, LED_SMD:LED_0603_1608Metric, F.Cu at (120.6, 44.2)
- added J302: Conn_01x02, Connector_JST:JST_PH_S2B-PH-K_1x02_P2.00mm_Horizontal, B.Cu at (128.2, 86.8)
- added L301: 2n9, Inductor_SMD:L_0402_1005Metric, F.Cu at (120.2, 50.6)
- added L302: 10u, Inductor_SMD:L_APV_ANR252012, F.Cu at (132.9, 48.4)
- added L303: 10u, Inductor_SMD:L_APV_ANR252012, F.Cu at (132.9, 55.2)
- added L304: 15n, Inductor_SMD:L_0603_1608Metric, F.Cu at (132.9, 57.6)
- added R317: 0R, Resistor_SMD:R_0402_1005Metric, F.Cu at (120.2, 48.4)
- added R318: 3k24, Resistor_SMD:R_0402_1005Metric, F.Cu at (138.6, 41.2)
- added R321: 33R, Resistor_SMD:R_0402_1005Metric, F.Cu at (120.8, 41.4)
- added R322: 10k, Resistor_SMD:R_0603_1608Metric, B.Cu at (91.4, 46.6)
- added R323: 10k, Resistor_SMD:R_0603_1608Metric, B.Cu at (99.4, 46.6)
- added R324: 10k, Resistor_SMD:R_0603_1608Metric, B.Cu at (107.2, 46.6)
- added R325: 10k, Resistor_SMD:R_0603_1608Metric, B.Cu at (115.0, 46.6)
- added R326: 10k, Resistor_SMD:R_0603_1608Metric, B.Cu at (138.8, 46.6)
- added R327: 10k, Resistor_SMD:R_0603_1608Metric, B.Cu at (146.6, 46.6)
- added R328: 10k, Resistor_SMD:R_0603_1608Metric, B.Cu at (154.6, 46.6)
- added R329: 10k, Resistor_SMD:R_0603_1608Metric, B.Cu at (162.6, 46.6)
- added R330: 10k, Resistor_SMD:R_0603_1608Metric, B.Cu at (170.2, 46.6)
- added R331: 10k, Resistor_SMD:R_0603_1608Metric, B.Cu at (83.6, 59.0)
- added R332: 10k, Resistor_SMD:R_0603_1608Metric, B.Cu at (91.4, 59.0)
- added R333: 10k, Resistor_SMD:R_0603_1608Metric, B.Cu at (99.4, 59.0)
- added R334: 10k, Resistor_SMD:R_0603_1608Metric, B.Cu at (107.2, 59.0)
- added R335: 10k, Resistor_SMD:R_0603_1608Metric, B.Cu at (115.0, 59.0)
- added R336: 10k, Resistor_SMD:R_0603_1608Metric, B.Cu at (138.8, 59.0)
- added R337: 10k, Resistor_SMD:R_0603_1608Metric, B.Cu at (146.6, 59.0)
- added R338: 10k, Resistor_SMD:R_0603_1608Metric, B.Cu at (154.6, 59.0)
- added R339: 10k, Resistor_SMD:R_0603_1608Metric, B.Cu at (162.6, 59.0)
- added R340: 10k, Resistor_SMD:R_0603_1608Metric, B.Cu at (170.2, 59.0)
- added R341: 10k, Resistor_SMD:R_0603_1608Metric, B.Cu at (83.6, 71.4)
- added R342: 10k, Resistor_SMD:R_0603_1608Metric, B.Cu at (91.4, 71.4)
- added R343: 10k, Resistor_SMD:R_0603_1608Metric, B.Cu at (99.4, 71.4)
- added R344: 10k, Resistor_SMD:R_0603_1608Metric, B.Cu at (107.2, 71.4)
- added R345: 10k, Resistor_SMD:R_0603_1608Metric, B.Cu at (115.0, 71.4)
- added R346: 10k, Resistor_SMD:R_0603_1608Metric, B.Cu at (138.8, 71.4)
- added R347: 10k, Resistor_SMD:R_0603_1608Metric, B.Cu at (146.6, 71.4)
- added R348: 10k, Resistor_SMD:R_0603_1608Metric, B.Cu at (154.6, 71.4)
- added R349: 10k, Resistor_SMD:R_0603_1608Metric, B.Cu at (162.6, 71.4)
- added R350: 10k, Resistor_SMD:R_0603_1608Metric, B.Cu at (170.2, 71.4)
- added R351: 10k, Resistor_SMD:R_0603_1608Metric, B.Cu at (99.4, 83.6)
- added R352: 10k, Resistor_SMD:R_0603_1608Metric, B.Cu at (107.2, 83.6)
- added R353: 10k, Resistor_SMD:R_0603_1608Metric, B.Cu at (115.0, 83.6)
- added R354: 10k, Resistor_SMD:R_0603_1608Metric, B.Cu at (138.8, 83.6)
- added R355: 10k, Resistor_SMD:R_0603_1608Metric, B.Cu at (146.6, 83.6)
- added R356: 10k, Resistor_SMD:R_0603_1608Metric, B.Cu at (154.6, 83.6)
- added U303: USBLC6-2P6, Package_TO_SOT_SMD:SOT-666, F.Cu at (127.0, 45.1)
- added U304: nRF52840, Package_DFN_QFN:Nordic_AQFN-73-1EP_7x7mm_P0.5mm, F.Cu at (126.8, 51.6)
- added U305: BQ24073RGT, Package_DFN_QFN:VQFN-16-1EP_3x3mm_P0.5mm_EP1.6x1.6mm, F.Cu at (135.8, 43.6)
- C201, C202, C312: footprint Capacitor_SMD:C_0603_1608Metric -> Capacitor_SMD:C_0402_1005Metric
- C304: value 1u -> 10u
- C306: value 100n -> 47n
- C307: value 100n -> 1u
- C308: value 100n -> 10u
- C309: value 100n -> 820p
- C310: value 100n -> 100p
- C313, C314: value 33p -> 12p
- R1, R2: footprint Resistor_SMD:R_0603_1608Metric -> Resistor_SMD:R_0402_1005Metric
- R301: value 27R -> 8k9
- R302: value 27R -> 10k
- R303: value 1k -> 10k; footprint Resistor_SMD:R_0402_1005Metric -> Resistor_SMD:R_0603_1608Metric; moved to B.Cu
- SW401, SW402, SW403, SW404, SW405, SW406, SW407, SW408, SW409, SW410, SW411, SW412, SW413, SW414, SW415, SW416, SW417, SW418, SW419, SW420, SW421, SW422, SW423, SW424, SW425, SW426, SW427, SW428, SW429, SW430, SW431, SW432, SW433, SW434, SW435, SW436: footprint Button_Switch_THT:SW_PUSH_6mm -> Button_Switch_THT:SW_PUSH_6mm_H7.3mm
- U201: value NCP1117-3.3_SOT223 -> XC6206PxxxMR; footprint Package_TO_SOT_SMD:SOT-223 -> Package_TO_SOT_SMD:SOT-23-3
- U301: value RP2040 -> TPS22914BYFPR; footprint Package_DFN_QFN:QFN-56-1EP_7x7mm_P0.4mm_EP3.2x3.2mm -> Package_BGA:Texas_PicoStar_BGA-4_0.758x0.758mm_Layout2x2_P0.4mm
- Y301: value 12MHz 20pF -> 32MHz 10p
- moved R303 51.2 mm to (83.6, 46.6), turned to 180 degrees
- moved J301 37.4 mm to (106.9, 41.6)
- moved U201 30.5 mm to (131.3, 64.0), turned to 0 degrees
- moved C201 30.0 mm to (134.0, 64.0)
- moved C202 24.3 mm to (128.6, 64.0), turned to 90 degrees
- moved C304 19.0 mm to (131.2, 46.1), turned to 0 degrees
- moved Y301 14.0 mm to (122.2, 59.4), turned to 180 degrees
- moved C305 13.3 mm to (132.1, 51.1)
- moved C313 12.1 mm to (121.4, 57.0), turned to 0 degrees
- moved R301 10.5 mm to (135.0, 40.8), turned to 180 degrees
- moved C311 10.4 mm to (132.6, 53.0), turned to 0 degrees
- moved C314 8.68 mm to (123.5, 57.0), turned to 180 degrees
- moved C308 7.01 mm to (129.2, 46.1), turned to 0 degrees
- moved C306 6.94 mm to (129.3, 57.4)
- moved R302 6.77 mm to (133.0, 42.5), turned to -90 degrees
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Connections:
- C201 pad 1: VBUS -> Net-(U201-VI)
- C301 pad 1: +1V1 -> VDD_NRF
- C302 pad 1: +1V1 -> VDD_NRF
- C303 pad 1: +1V1 -> VDD_NRF
- C304 pad 1: +3V3 -> VBUS
- C305 pad 1: +3V3 -> VDD_NRF
- C306 pad 1: +3V3 -> Net-(U304-DEC4)
- C307 pad 1: +3V3 -> Net-(U304-DEC4)
- C308 pad 1: +3V3 -> Net-(U304-DECUSB)
- C309 pad 1: +3V3 -> Net-(U304-DEC5)
- C310 pad 1: +3V3 -> Net-(U304-DEC3)
- C311 pad 1: +3V3 -> Net-(U304-DEC1)
- C312 pad 1: +3V3 -> VDD_NRF
- C313 pad 2: Net-(U301-XIN) -> Net-(U304-XC1)
- C314 pad 2: Net-(U301-XOUT) -> Net-(U304-XC2)
- J1 pad A6: /Microcontroller/USB_DP -> /USB_CON_DP
- J1 pad A7: /Microcontroller/USB_DN -> /USB_CON_DN
- J1 pad B6: /Microcontroller/USB_DP -> /USB_CON_DP
- J1 pad B7: /Microcontroller/USB_DN -> /USB_CON_DN
- R301 pad 1: Net-(U301-USB_DP) -> GND
- R301 pad 2: /Microcontroller/USB_DP -> Net-(U305-ISET)
- R302 pad 1: Net-(U301-USB_DM) -> GND
- R302 pad 2: /Microcontroller/USB_DN -> Net-(U305-TS)
- R303 pad 1: /Microcontroller/QSPI_SS -> VDD_NRF
- R303 pad 2: /Microcontroller/~{USB_BOOT} -> BTN0_0
- SW401 pad 1: /Keyboard Matrix/COL0 -> BTN0_0
- SW401 pad 2: Net-(D401-A) -> GND
- SW402 pad 1: /Keyboard Matrix/COL1 -> BTN0_1
- SW402 pad 2: Net-(D402-A) -> GND
- SW403 pad 1: /Keyboard Matrix/COL2 -> BTN0_2
- SW403 pad 2: Net-(D403-A) -> GND
- SW404 pad 1: /Keyboard Matrix/COL3 -> BTN0_3
- SW404 pad 2: Net-(D404-A) -> GND
- SW405 pad 1: /Keyboard Matrix/COL4 -> BTN0_4
- SW405 pad 2: Net-(D405-A) -> GND
- SW406 pad 1: /Keyboard Matrix/COL5 -> BTN0_5
- SW406 pad 2: Net-(D406-A) -> GND
- SW407 pad 1: /Keyboard Matrix/COL6 -> BTN0_6
- SW407 pad 2: Net-(D407-A) -> GND
- SW408 pad 1: /Keyboard Matrix/COL7 -> BTN0_7
- SW408 pad 2: Net-(D408-A) -> GND
- SW409 pad 1: /Keyboard Matrix/COL8 -> BTN0_8
- SW409 pad 2: Net-(D409-A) -> GND
- SW410 pad 1: /Keyboard Matrix/COL9 -> BTN0_9
- SW410 pad 2: Net-(D410-A) -> GND
- SW411 pad 1: /Keyboard Matrix/COL0 -> BTN1_0
- SW411 pad 2: Net-(D411-A) -> GND
- SW412 pad 1: /Keyboard Matrix/COL1 -> BTN1_1
- SW412 pad 2: Net-(D412-A) -> GND
- SW413 pad 1: /Keyboard Matrix/COL2 -> BTN1_2
- SW413 pad 2: Net-(D413-A) -> GND
- SW414 pad 1: /Keyboard Matrix/COL3 -> BTN1_3
- SW414 pad 2: Net-(D414-A) -> GND
- SW415 pad 1: /Keyboard Matrix/COL4 -> BTN1_4
- SW415 pad 2: Net-(D415-A) -> GND
- SW416 pad 1: /Keyboard Matrix/COL5 -> BTN1_5
- SW416 pad 2: Net-(D416-A) -> GND
- SW417 pad 1: /Keyboard Matrix/COL6 -> BTN1_6
- SW417 pad 2: Net-(D417-A) -> GND
- SW418 pad 1: /Keyboard Matrix/COL7 -> BTN1_7
- SW418 pad 2: Net-(D418-A) -> GND
- SW419 pad 1: /Keyboard Matrix/COL8 -> BTN1_8
- SW419 pad 2: Net-(D419-A) -> GND
- SW420 pad 1: /Keyboard Matrix/COL9 -> BTN1_9
- SW420 pad 2: Net-(D420-A) -> GND
- SW421 pad 1: /Keyboard Matrix/COL0 -> BTN2_0
- SW421 pad 2: Net-(D421-A) -> GND
- SW422 pad 1: /Keyboard Matrix/COL1 -> BTN2_1
- SW422 pad 2: Net-(D422-A) -> GND
- SW423 pad 1: /Keyboard Matrix/COL2 -> BTN2_2
- SW423 pad 2: Net-(D423-A) -> GND
- SW424 pad 1: /Keyboard Matrix/COL3 -> BTN2_3
- SW424 pad 2: Net-(D424-A) -> GND
- SW425 pad 1: /Keyboard Matrix/COL4 -> BTN2_4
- SW425 pad 2: Net-(D425-A) -> GND
- SW426 pad 1: /Keyboard Matrix/COL5 -> BTN2_5
- SW426 pad 2: Net-(D426-A) -> GND
- SW427 pad 1: /Keyboard Matrix/COL6 -> BTN2_6
- SW427 pad 2: Net-(D427-A) -> GND
- SW428 pad 1: /Keyboard Matrix/COL7 -> BTN2_7
- SW428 pad 2: Net-(D428-A) -> GND
- SW429 pad 1: /Keyboard Matrix/COL8 -> BTN2_8
- SW429 pad 2: Net-(D429-A) -> GND
- SW430 pad 1: /Keyboard Matrix/COL9 -> BTN2_9
- SW430 pad 2: Net-(D430-A) -> GND
- SW431 pad 1: /Keyboard Matrix/COL2 -> BTN3_0
- SW431 pad 2: Net-(D431-A) -> GND
- SW432 pad 1: /Keyboard Matrix/COL3 -> BTN3_1
- SW432 pad 2: Net-(D432-A) -> GND
- SW433 pad 1: /Keyboard Matrix/COL4 -> BTN3_2
- SW433 pad 2: Net-(D433-A) -> GND
- SW434 pad 1: /Keyboard Matrix/COL5 -> BTN3_3
- SW434 pad 2: Net-(D434-A) -> GND
- SW435 pad 1: /Keyboard Matrix/COL6 -> BTN3_4
- SW435 pad 2: Net-(D435-A) -> GND
- SW436 pad 1: /Keyboard Matrix/COL7 -> BTN3_5
- SW436 pad 2: Net-(D436-A) -> GND
- U201 pad 3: VBUS -> Net-(U201-VI)
- Y301 pad 1: Net-(U301-XOUT) -> Net-(U304-XC2)
- Y301 pad 3: Net-(U301-XIN) -> Net-(U304-XC1)
Routing:
- net +3V3: track 223.8 -> 0.00 mm, vias 29 -> 0
- net Net-(Q301-D): track 176.9 -> 0.00 mm
- net /Keyboard Matrix/ROW2: track 175.1 -> 0.00 mm, vias 2 -> 0
- net /Keyboard Matrix/ROW0: track 170.0 -> 0.00 mm, vias 2 -> 0
- net /Keyboard Matrix/ROW1: track 158.1 -> 0.00 mm, vias 2 -> 0
- net /Keyboard Matrix/ROW3: track 130.8 -> 0.00 mm, vias 1 -> 0
- net /Keyboard Matrix/COL0: track 78.1 -> 0.00 mm
- net /Keyboard Matrix/COL9: track 73.9 -> 0.00 mm
- net /Keyboard Matrix/COL2: track 73.4 -> 0.00 mm
- net /Keyboard Matrix/COL1: track 69.3 -> 0.00 mm
- net /Keyboard Matrix/COL7: track 69.1 -> 0.00 mm
- net LED_SW: track 66.4 -> 0.00 mm, vias 2 -> 0
- net /Keyboard Matrix/COL3: track 65.4 -> 0.00 mm
- net /Keyboard Matrix/COL8: track 65.1 -> 0.00 mm
- net /Keyboard Matrix/COL6: track 60.9 -> 0.00 mm
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- removed copper zone on F.Cu, net +3V3
- removed copper zone on In2.Cu, net +3V3
- removed copper zone on B.Cu, net GND
- removed copper zone on F.Cu, net GND
- removed copper zone on In1.Cu, net GND
- removed copper zone on In2.Cu, net GND
Other:
- outline, holes or cut-outs redrawn
- board text removed: "DESIGNED BY @SINI6A"

Commit message: board routed
Parts:
- removed R322, R323, R324, R325, R326, R327, R328, R329, R330, R331, R332, R333, R334, R335, R336, R337, R338, R339, R340, R341, R342, R343, R344, R345, R346, R347, R348, R349, R350, R351, R352, R353, R354, R355, R356: 10k, Resistor_SMD:R_0603_1608Metric
- added AE301: Antenna, mikoto:2.4GHz-meander-antenna-v2-inverted, F.Cu at (105.8, 41.9)
- added C321: 100n, Capacitor_SMD:C_0402_1005Metric, F.Cu at (135.0, 39.6)
- added D401: D, Diode_SMD:D_SOD-123, B.Cu at (84.1, 52.1)
- added D402: D, Diode_SMD:D_SOD-123, B.Cu at (92.0, 52.1)
- added D403: D, Diode_SMD:D_SOD-123, B.Cu at (99.9, 52.1)
- added D404: D, Diode_SMD:D_SOD-123, B.Cu at (107.6, 52.1)
- added D405: D, Diode_SMD:D_SOD-123, B.Cu at (115.6, 52.1)
- added D406: D, Diode_SMD:D_SOD-123, B.Cu at (139.5, 52.1)
- added D407: D, Diode_SMD:D_SOD-123, B.Cu at (147.4, 52.1)
- added D408: D, Diode_SMD:D_SOD-123, B.Cu at (155.2, 52.1)
- added D409: D, Diode_SMD:D_SOD-123, B.Cu at (163.1, 52.1)
- added D411: D, Diode_SMD:D_SOD-123, B.Cu at (84.1, 64.5)
- added D412: D, Diode_SMD:D_SOD-123, B.Cu at (92.0, 64.5)
- added D413: D, Diode_SMD:D_SOD-123, B.Cu at (99.9, 64.5)
- added D414: D, Diode_SMD:D_SOD-123, B.Cu at (107.8, 64.5)
- added D415: D, Diode_SMD:D_SOD-123, B.Cu at (115.6, 64.5)
- added D416: D, Diode_SMD:D_SOD-123, B.Cu at (139.5, 64.5)
- added D417: D, Diode_SMD:D_SOD-123, B.Cu at (147.4, 64.5)
- added D418: D, Diode_SMD:D_SOD-123, B.Cu at (155.2, 64.5)
- added D419: D, Diode_SMD:D_SOD-123, B.Cu at (163.2, 64.5)
- added D420: D, Diode_SMD:D_SOD-123, B.Cu at (171.0, 64.5)
- added D421: D, Diode_SMD:D_SOD-123, B.Cu at (84.1, 77.0)
- added D422: D, Diode_SMD:D_SOD-123, B.Cu at (92.0, 77.0)
- added D423: D, Diode_SMD:D_SOD-123, B.Cu at (99.9, 77.0)
- added D424: D, Diode_SMD:D_SOD-123, B.Cu at (107.8, 77.0)
- added D425: D, Diode_SMD:D_SOD-123, B.Cu at (115.6, 77.0)
- added D426: D, Diode_SMD:D_SOD-123, B.Cu at (139.5, 77.0)
- added D427: D, Diode_SMD:D_SOD-123, B.Cu at (147.4, 77.0)
- added D428: D, Diode_SMD:D_SOD-123, B.Cu at (155.2, 77.0)
- added D429: D, Diode_SMD:D_SOD-123, B.Cu at (163.1, 77.0)
- added D430: D, Diode_SMD:D_SOD-123, B.Cu at (171.0, 77.0)
- added D431: D, Diode_SMD:D_SOD-123, B.Cu at (99.9, 89.2)
- added D432: D, Diode_SMD:D_SOD-123, B.Cu at (107.8, 89.2)
- added D433: D, Diode_SMD:D_SOD-123, B.Cu at (115.6, 89.2)
- added D434: D, Diode_SMD:D_SOD-123, B.Cu at (139.5, 89.2)
- added D435: D, Diode_SMD:D_SOD-123, B.Cu at (147.4, 89.2)
- added D436: D, Diode_SMD:D_SOD-123, B.Cu at (155.2, 89.2)
- added JP301: Jumper_2_Open, Jumper:SolderJumper-2_P1.3mm_Open_RoundedPad1.0x1.5mm, F.Cu at (149.8, 42.0)
- added SW301: SW_SPST, Button_Switch_SMD:SW_SPDT_PCM12, F.Cu at (148.2, 37.4)
- added U302: MAX17048, Pocketboard:21-0555B_W80B1-1_MXM, F.Cu at (134.9, 37.9)
- J302: footprint Connector_JST:JST_PH_S2B-PH-K_1x02_P2.00mm_Horizontal -> Connector_PinSocket_2.54mm:PinSocket_1x02_P2.54mm_Vertical
- R301: value 8k9 -> 10k
- R303: footprint Resistor_SMD:R_0603_1608Metric -> Resistor_SMD:R_0402_1005Metric; moved to F.Cu
- SW401, SW402, SW403, SW404, SW405, SW406, SW407, SW408, SW409, SW410, SW411, SW412, SW413, SW414, SW415, SW416, SW417, SW418, SW419, SW420, SW421, SW422, SW423, SW424, SW425, SW426, SW427, SW428, SW429, SW430, SW431, SW432, SW433, SW434, SW435, SW436: footprint Button_Switch_THT:SW_PUSH_6mm_H7.3mm -> Button_Switch_THT:SW_PUSH_6mm
- moved R303 59.3 mm to (142.8, 45.4), turned to -90 degrees
- moved J301 23.9 mm to (83.2, 44.9)
- moved C319 19.5 mm to (139.8, 43.3), turned to 90 degrees
- moved U301 17.2 mm to (140.8, 45.8), turned to 0 degrees
- moved C320 14.1 mm to (138.2, 46.7), turned to 180 degrees
- moved R317 7.54 mm to (116.3, 41.9), turned to 0 degrees
- moved R2 7.24 mm to (124.7, 44.1), turned to 0 degrees
- moved C317 7.20 mm to (116.2, 40.9)
- moved R1 7.16 mm to (129.2, 44.1), turned to 180 degrees
- moved C202 5.45 mm to (132.7, 67.7), turned to 180 degrees
- moved C302 3.33 mm to (132.4, 54.6), turned to 0 degrees
- moved C201 2.81 mm to (131.7, 62.4), turned to 180 degrees
- moved L303 2.80 mm to (132.9, 58.0)
- moved L304 2.28 mm to (130.7, 58.0), turned to 90 degrees
- moved U201 1.40 mm to (132.2, 65.0), turned to 90 degrees
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Connections:
- net ANTENNA renamed Net-(AE301-A)
- net Net-(J302-Pin_1) renamed /Power/VBAT
- C201 pad 1: Net-(U201-VI) -> /Microcontroller/VDDH
- C204 pad 1: /Microcontroller/VDDH -> Net-(JP301-B)
- C319 pad 1: /Microcontroller/VDDH -> Net-(JP301-B)
- C320 pad 1: Net-(U201-VI) -> /Microcontroller/VDDH
- J301 pad 1: +3V3 -> VDD_NRF
- R303 pad 1: VDD_NRF -> GND
- R303 pad 2: BTN0_0 -> Net-(JP301-A)
- SW401 pad 1: BTN0_0 -> /Keyboard Matrix/COL0
- SW401 pad 2: GND -> Net-(D401-A)
- SW402 pad 1: BTN0_1 -> /Keyboard Matrix/COL1
- SW402 pad 2: GND -> Net-(D402-A)
- SW403 pad 1: BTN0_2 -> /Keyboard Matrix/COL2
- SW403 pad 2: GND -> Net-(D403-A)
- SW404 pad 1: BTN0_3 -> /Keyboard Matrix/COL3
- SW404 pad 2: GND -> Net-(D404-A)
- SW405 pad 1: BTN0_4 -> /Keyboard Matrix/COL4
- SW405 pad 2: GND -> Net-(D405-A)
- SW406 pad 1: BTN0_5 -> /Keyboard Matrix/COL5
- SW406 pad 2: GND -> Net-(D406-A)
- SW407 pad 1: BTN0_6 -> /Keyboard Matrix/COL6
- SW407 pad 2: GND -> Net-(D407-A)
- SW408 pad 1: BTN0_7 -> /Keyboard Matrix/COL7
- SW408 pad 2: GND -> Net-(D408-A)
- SW409 pad 1: BTN0_8 -> /Keyboard Matrix/COL8
- SW409 pad 2: GND -> Net-(D409-A)
- SW410 pad 1: BTN0_9 -> /Keyboard Matrix/P_BTN
- SW411 pad 1: BTN1_0 -> /Keyboard Matrix/COL0
- SW411 pad 2: GND -> Net-(D411-A)
- SW412 pad 1: BTN1_1 -> /Keyboard Matrix/COL1
- SW412 pad 2: GND -> Net-(D412-A)
- SW413 pad 1: BTN1_2 -> /Keyboard Matrix/COL2
- SW413 pad 2: GND -> Net-(D413-A)
- SW414 pad 1: BTN1_3 -> /Keyboard Matrix/COL3
- SW414 pad 2: GND -> Net-(D414-A)
- SW415 pad 1: BTN1_4 -> /Keyboard Matrix/COL4
- SW415 pad 2: GND -> Net-(D415-A)
- SW416 pad 1: BTN1_5 -> /Keyboard Matrix/COL5
- SW416 pad 2: GND -> Net-(D416-A)
- SW417 pad 1: BTN1_6 -> /Keyboard Matrix/COL6
- SW417 pad 2: GND -> Net-(D417-A)
- SW418 pad 1: BTN1_7 -> /Keyboard Matrix/COL7
- SW418 pad 2: GND -> Net-(D418-A)
- SW419 pad 1: BTN1_8 -> /Keyboard Matrix/COL8
- SW419 pad 2: GND -> Net-(D419-A)
- SW420 pad 1: BTN1_9 -> /Keyboard Matrix/COL9
- SW420 pad 2: GND -> Net-(D420-A)
- SW421 pad 1: BTN2_0 -> /Keyboard Matrix/COL0
- SW421 pad 2: GND -> Net-(D421-A)
- SW422 pad 1: BTN2_1 -> /Keyboard Matrix/COL1
- SW422 pad 2: GND -> Net-(D422-A)
- SW423 pad 1: BTN2_2 -> /Keyboard Matrix/COL2
- SW423 pad 2: GND -> Net-(D423-A)
- SW424 pad 1: BTN2_3 -> /Keyboard Matrix/COL3
- SW424 pad 2: GND -> Net-(D424-A)
- SW425 pad 1: BTN2_4 -> /Keyboard Matrix/COL4
- SW425 pad 2: GND -> Net-(D425-A)
- SW426 pad 1: BTN2_5 -> /Keyboard Matrix/COL5
- SW426 pad 2: GND -> Net-(D426-A)
- SW427 pad 1: BTN2_6 -> /Keyboard Matrix/COL6
- SW427 pad 2: GND -> Net-(D427-A)
- SW428 pad 1: BTN2_7 -> /Keyboard Matrix/COL7
- SW428 pad 2: GND -> Net-(D428-A)
- SW429 pad 1: BTN2_8 -> /Keyboard Matrix/COL8
- SW429 pad 2: GND -> Net-(D429-A)
- SW430 pad 1: BTN2_9 -> /Keyboard Matrix/COL9
- SW430 pad 2: GND -> Net-(D430-A)
- SW431 pad 1: BTN3_0 -> /Keyboard Matrix/COL2
- SW431 pad 2: GND -> Net-(D431-A)
- SW432 pad 1: BTN3_1 -> /Keyboard Matrix/COL3
- SW432 pad 2: GND -> Net-(D432-A)
- SW433 pad 1: BTN3_2 -> /Keyboard Matrix/COL4
- SW433 pad 2: GND -> Net-(D433-A)
- SW434 pad 1: BTN3_3 -> /Keyboard Matrix/COL5
- SW434 pad 2: GND -> Net-(D434-A)
- SW435 pad 1: BTN3_4 -> /Keyboard Matrix/COL6
- SW435 pad 2: GND -> Net-(D435-A)
- SW436 pad 1: BTN3_5 -> /Keyboard Matrix/COL7
- SW436 pad 2: GND -> Net-(D436-A)
- U201 pad 3: Net-(U201-VI) -> /Microcontroller/VDDH
- U301 pad A1: Net-(U201-VI) -> /Microcontroller/VDDH
- U301 pad A2: /Microcontroller/VDDH -> Net-(JP301-B)
- U301 pad B2: LCD_PWR -> Net-(JP301-A)
- U304 pad A10: /LCD/~{CS} -> unconnected-(U304-AIN5/P0.29-PadA10)
- U304 pad A14: unconnected-(U304-P1.15-PadA14) -> /LCD/D/C
- U304 pad A16: unconnected-(U304-P1.13-PadA16) -> /LCD/~{CS}
- U304 pad A20: BTN3_4 -> unconnected-(U304-P1.10-PadA20)
- U304 pad A8: BTN2_3 -> unconnected-(U304-AIN7/P0.31-PadA8)
- U304 pad AC11: BTN1_1 -> unconnected-(U304-P0.16-PadAC11)
- U304 pad AC15: BTN1_3 -> unconnected-(U304-P0.19-PadAC15)
- U304 pad AC17: BTN1_5 -> unconnected-(U304-P0.21-PadAC17)
- U304 pad AC19: BTN1_7 -> unconnected-(U304-P0.23-PadAC19)
- U304 pad AC21: BTN1_9 -> unconnected-(U304-P0.25-PadAC21)
- U304 pad AC9: BTN1_0 -> unconnected-(U304-P0.14-PadAC9)
- U304 pad AD12: BTN1_2 -> unconnected-(U304-P0.17-PadAD12)
- U304 pad AD16: BTN1_4 -> unconnected-(U304-P0.20-PadAD16)
- U304 pad AD18: BTN1_6 -> unconnected-(U304-P0.22-PadAD18)
- U304 pad AD20: BTN1_8 -> unconnected-(U304-P0.24-PadAD20)
- U304 pad AD22: BTN2_4 -> unconnected-(U304-TRACEDATA0/P1.00-PadAD22)
- U304 pad AD8: BTN0_9 -> unconnected-(U304-P0.13-PadAD8)
- U304 pad B11: BTN2_1 -> /Keyboard Matrix/ROW3
- U304 pad B15: unconnected-(U304-P1.14-PadB15) -> /LCD/~{RESET}
- U304 pad B17: LCD_PWR -> /Keyboard Matrix/ROW2
- U304 pad B19: BTN3_5 -> /Keyboard Matrix/ROW1
- U304 pad B9: BTN2_2 -> unconnected-(U304-AIN6/P0.30-PadB9)
- U304 pad D2: BTN0_0 -> unconnected-(U304-XL1/P0.00-PadD2)
- U304 pad F2: BTN0_1 -> unconnected-(U304-XL2/P0.01-PadF2)
- U304 pad G1: LED_SW -> /Keyboard Matrix/COL9
- U304 pad H2: BTN2_0 -> unconnected-(U304-P0.27-PadH2)
- U304 pad J1: /LCD/~{RESET} -> /Keyboard Matrix/P_BTN
- U304 pad J24: BTN0_6 -> unconnected-(U304-NFC2/P0.10-PadJ24)
- U304 pad K2: /LCD/D/C -> unconnected-(U304-AIN3/P0.05-PadK2)
- U304 pad L1: BTN0_3 -> /Keyboard Matrix/COL8
- U304 pad L24: BTN0_5 -> /Keyboard Matrix/COL0
- U304 pad M2: BTN0_4 -> BAT_I2C_SCL
- U304 pad N1: BTN0_2 -> /Keyboard Matrix/COL7
- U304 pad P2: BTN3_2 -> unconnected-(U304-P1.08-PadP2)
- U304 pad P23: BTN3_1 -> /Keyboard Matrix/COL1
- U304 pad R1: BTN3_3 -> /Keyboard Matrix/COL6
- U304 pad R24: BTN3_0 -> /Keyboard Matrix/COL2
- U304 pad T2: BTN0_7 -> BAT_I2C_SDA
- U304 pad T23: BTN2_9 -> unconnected-(U304-P1.05-PadT23)
- U304 pad U1: BTN0_8 -> /Keyboard Matrix/COL5
- U304 pad U24: BTN2_8 -> /Keyboard Matrix/COL3
- U304 pad V23: BTN2_7 -> unconnected-(U304-P1.03-PadV23)
- U304 pad W24: BTN2_6 -> /Keyboard Matrix/COL4
- U304 pad Y23: BTN2_5 -> /Keyboard Matrix/ROW0
- U305 pad 10: /Microcontroller/VDDH -> Net-(JP301-B)
- U305 pad 11: /Microcontroller/VDDH -> Net-(JP301-B)
- U305 pad 6: /Microcontroller/VDDH -> Net-(JP301-B)
Routing:
- net /Keyboard Matrix/ROW2: track 0.00 -> 134.8 mm, vias 0 -> 3
- net /Keyboard Matrix/ROW0: track 0.00 -> 134.5 mm, vias 0 -> 3
- net /Keyboard Matrix/ROW1: track 0.00 -> 121.2 mm, vias 0 -> 3
- net /Keyboard Matrix/ROW3: track 0.00 -> 107.7 mm, vias 0 -> 1
- net /Keyboard Matrix/COL0: track 0.00 -> 75.4 mm, vias 0 -> 2
- net /Keyboard Matrix/COL2: track 0.00 -> 71.5 mm, vias 0 -> 2
- net /Keyboard Matrix/COL7: track 0.00 -> 68.6 mm
- net /Keyboard Matrix/COL1: track 0.00 -> 67.8 mm, vias 0 -> 2
- net /Power/VBAT: track 0.00 -> 65.3 mm, vias 0 -> 3
- net /Keyboard Matrix/COL8: track 0.00 -> 64.2 mm
- net /Keyboard Matrix/COL9: track 0.00 -> 63.7 mm
- net /Keyboard Matrix/COL3: track 0.00 -> 63.5 mm, vias 0 -> 2
- net /Keyboard Matrix/COL6: track 0.00 -> 60.4 mm
- net /Keyboard Matrix/COL4: track 0.00 -> 55.4 mm, vias 0 -> 2
- net GND: track 0.00 -> 53.8 mm, vias 0 -> 188
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- added copper zone on In2.Cu, net /Microcontroller/VDDH
- added copper zone on B.Cu, net GND
- added copper zone on F.Cu, net GND
- added copper zone on In1.Cu, net GND
- added copper zone on In2.Cu, net VBUS
- added copper zone on In2.Cu, net VDD_NRF
Other:
- outline, holes or cut-outs redrawn
- board text added: "JLC calculator gives 0.4983mm trace width, with 0.125mm separation for 04161H-7628 stackup"
- board text removed: "<"
- board text removed: "?"
- board text removed: "A"
- board text removed: "B"
- board text removed: "C"
- board text removed: "D"
- board text removed: "E"
- board text removed: "G"
- board text removed: "H"
- board text removed: "I"
- board text removed: "K"
- board text removed: "N"
- board text removed: "O"
- board text removed: "P"
- board text removed: "Q"
- board text removed: "R"
- board text removed: "T"
- board text removed: "U"
- board text removed: "USB BOOT"
- board text removed: "W"
- board text removed: "Z"
- board text removed: "del"
- board text removed: "ent"
- board text removed: "esc"
- board text removed: "tab"
- board text removed: "‘"
